File: connectors.kicad_sch (KiCad schematic)
At the start: 2 parts, among them J1 USB_C_Receptacle_USB2.0_14P, J2 Conn_01x02_Socket

Commit message: Remove 12V buck converter and power rail
Parts:
- removed J2: Conn_01x02_Socket, symbol Connector:Conn_01x02_Socket
Other:
- note removed: "External 12V Socket"
Changed lines of the file:
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@@
-    (stroke (width 0) (type default))
-  )
-  (wire (pts (xy 118.11 34.29) (xy 118.11 38.1))
     (stroke (width 0) (type default))
   )
@@
     (stroke (width 0) (type default))
   )
-  (wire (pts (xy 118.11 27.94) (xy 118.11 31.75))
-    (stroke (width 0) (type default))
-  )
-  (wire (pts (xy 118.11 34.29) (xy 127 34.29))
-    (stroke (width 0) (type default))
-  )
   (wire (pts (xy 245.11 50.8) (xy 254 50.8))
     (stroke (width 0) (type default))
@@
   )
   (wire (pts (xy 68.58 49.53) (xy 68.58 52.07))
-    (stroke (width 0) (type default))
-  )
-  (wire (pts (xy 118.11 31.75) (xy 127 31.75))
     (stroke (width 0) (type default))
   )
@@
   (text "Only ground shield\non host side" (at 40.64 69.85 0)
     (effects (font (size 1.27 1.27)) (justify right bottom))
-  )
-  (text "External 12V Socket" (at 127 27.94 0)
-    (effects (font (size 1.27 1.27)) (justify left bottom))
   )
   (label "VBUS" (at 80.01 31.75 180) (fields_autoplaced)
@@
     (effects (font (size 1.27 1.27)) (justify left))
   )
-  (symbol (lib_id "power:+12V") (at 118.11 27.94 0) (unit 1)
-    (in_bom yes) (on_board yes) (dnp no) (fields_autoplaced)
-    (property "Reference" "#PWR050" (at 118.11 31.75 0)
-      (effects (font (size 1.27 1.27)) hide)
-    )
-    (property "Value" "+12V" (at 118.11 22.86 0)
-      (effects (font (size 1.27 1.27)))
-    )
-    (property "Footprint" "" (at 118.11 27.94 0)
-      (effects (font (size 1.27 1.27)) hide)
-    )
-    (property "Datasheet" "" (at 118.11 27.94 0)
-      (effects (font (size 1.27 1.27)) hide)
-    )
-    (pin "1")
-    (instances
-      (project "mainboard"
-        (path "/613f8c39-c37c-4981-8911-5138d36a7959/d53978c6-3f4c-472f-b8a8-1027880c9a69"
-          (reference "#PWR050") (unit 1)
-        )
-      )
-    )
-  )
   (symbol (lib_id "power:GND") (at 245.11 57.15 0) (unit 1)
     (in_bom yes) (on_board yes) (dnp no) (fields_autoplaced)
@@
     )
   )
-  (symbol (lib_id "Connector:Conn_01x02_Socket") (at 132.08 31.75 0) (unit 1)
-    (in_bom yes) (on_board yes) (dnp no) (fields_autoplaced)
-    (property "Reference" "J2" (at 133.35 31.75 0)
-      (effects (font (size 1.27 1.27)) (justify left))
-    )
-    (property "Value" "Conn_01x02_Socket" (at 133.35 34.29 0)
-      (effects (font (size 1.27 1.27)) (justify left))
-    )
-    (property "Footprint" "" (at 132.08 31.75 0)
-      (effects (font (size 1.27 1.27)) hide)
-    )
-    (property "Datasheet" "~" (at 132.08 31.75 0)
-      (effects (font (size 1.27 1.27)) hide)
-    )
-    (pin "2")
-    (pin "1")
-    (instances
-      (project "mainboard"
-        (path "/613f8c39-c37c-4981-8911-5138d36a7959/d53978c6-3f4c-472f-b8a8-1027880c9a69"
-          (reference "J2") (unit 1)
-        )
-      )
-    )
-  )
   (symbol (lib_id "Connector:USB_C_Receptacle_USB2.0_14P") (at 53.34 46.99 0) (unit 1)
     (in_bom yes) (on_board yes) (dnp no) (fields_autoplaced)
@@
         )
       )
-    )
-  )
-  (symbol (lib_id "power:GND") (at 118.11 38.1 0) (unit 1)
-    (in_bom yes) (on_board yes) (dnp no) (fields_autoplaced)
-    (property "Reference" "#PWR051" (at 118.11 44.45 0)
-      (effects (font (size 1.27 1.27)) hide)
-    )
-    (property "Value" "GND" (at 118.11 43.18 0)
-      (effects (font (size 1.27 1.27)))
-    )
-    (property "Footprint" "" (at 118.11 38.1 0)
-      (effects (font (size 1.27 1.27)) hide)
-    )
-    (property "Datasheet" "" (at 118.11 38.1 0)
-      (effects (font (size 1.27 1.27)) hide)
-    )
-    (pin "1")
-    (instances
-      (project "mainboard"
-        (path "/613f8c39-c37c-4981-8911-5138d36a7959/d53978c6-3f4c-472f-b8a8-1027880c9a69"
-          (reference "#PWR051") (unit 1)
-        )
-      )
