File: motor_control.kicad_sch (KiCad schematic)
At the start: 9 parts, among them Q8 IRLML2502, U2 DRV8870DDAR

Commit message: Reannotate geographically by layout
Parts:
- renumbered C2 to C1, C5 to C2, R2 to R1, R19 to R17, R3 to R2, U2 to U1
Changed lines of the file:
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@@
   (symbol (lib_id "Device:R") (at 190.5 99.06 90) (unit 1)
     (in_bom yes) (on_board yes) (dnp no) (fields_autoplaced)
-    (property "Reference" "R3" (at 190.5 92.71 90)
+    (property "Reference" "R2" (at 190.5 92.71 90)
       (effects (font (size 1.27 1.27)))
     )
@@
       (project "mainboard"
         (path "/613f8c39-c37c-4981-8911-5138d36a7959/ecb72cc6-9992-49a0-afcf-3c2905614ae7"
-          (reference "R3") (unit 1)
+          (reference "R2") (unit 1)
         )
       )
@@
   (symbol (lib_id "Driver_Motor:DRV8870DDA") (at 115.57 99.06 0) (unit 1)
     (in_bom yes) (on_board yes) (dnp no) (fields_autoplaced)
-    (property "Reference" "U2" (at 117.7641 88.9 0)
+    (property "Reference" "U1" (at 117.7641 88.9 0)
       (effects (font (size 1.27 1.27)) (justify left))
     )
@@
       (project "mainboard"
         (path "/613f8c39-c37c-4981-8911-5138d36a7959/ecb72cc6-9992-49a0-afcf-3c2905614ae7"
-          (reference "U2") (unit 1)
+          (reference "U1") (unit 1)
         )
       )
@@
   (symbol (lib_id "Device:C_Polarized") (at 102.87 76.2 0) (unit 1)
     (in_bom yes) (on_board yes) (dnp no) (fields_autoplaced)
-    (property "Reference" "C5" (at 106.68 74.041 0)
+    (property "Reference" "C2" (at 106.68 74.041 0)
       (effects (font (size 1.27 1.27)) (justify left))
     )
@@
       (project "mainboard"
         (path "/613f8c39-c37c-4981-8911-5138d36a7959/ecb72cc6-9992-49a0-afcf-3c2905614ae7"
-          (reference "C5") (unit 1)
+          (reference "C2") (unit 1)
         )
       )
@@
   (symbol (lib_id "Device:R") (at 133.35 110.49 0) (unit 1)
     (in_bom yes) (on_board yes) (dnp no) (fields_autoplaced)
-    (property "Reference" "R2" (at 135.89 109.22 0)
+    (property "Reference" "R1" (at 135.89 109.22 0)
       (effects (font (size 1.27 1.27)) (justify left))
     )
@@
       (project "mainboard"
         (path "/613f8c39-c37c-4981-8911-5138d36a7959/ecb72cc6-9992-49a0-afcf-3c2905614ae7"
-          (reference "R2") (unit 1)
+          (reference "R1") (unit 1)
         )
       )
@@
   (symbol (lib_id "Device:C") (at 88.9 76.2 0) (mirror y) (unit 1)
     (in_bom yes) (on_board yes) (dnp no)
-    (property "Reference" "C2" (at 85.09 74.93 0)
+    (property "Reference" "C1" (at 85.09 74.93 0)
       (effects (font (size 1.27 1.27)) (justify left))
     )
@@
       (project "mainboard"
         (path "/613f8c39-c37c-4981-8911-5138d36a7959/ecb72cc6-9992-49a0-afcf-3c2905614ae7"
-          (reference "C2") (unit 1)
+          (reference "C1") (unit 1)
         )
       )
@@
   (symbol (lib_id "Device:R") (at 210.185 108.585 0) (unit 1)
     (in_bom yes) (on_board yes) (dnp no) (fields_autoplaced)
-    (property "Reference" "R19" (at 212.725 107.315 0)
+    (property "Reference" "R17" (at 212.725 107.315 0)
       (effects (font (size 1.27 1.27)) (justify left))
     )
@@
       (project "mainboard"
         (path "/613f8c39-c37c-4981-8911-5138d36a7959/ecb72cc6-9992-49a0-afcf-3c2905614ae7"
-          (reference "R19") (unit 1)
-        )
-      )
+          (reference "R17") (unit 1)
+        )
+      )

Commit message: Fix revision
Other:
- title: openautolab - Mainboard -> openautolab - Alternative Mainboard
Changed lines of the file:
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@@
   (paper "A4")
   (title_block
-    (title "openautolab - Mainboard")
+    (title "openautolab - Alternative Mainboard")
     (date "2024-04-03")
-    (rev "2.0")
+    (rev "1")
   )
   (junction (at 210.185 99.06) (diameter 0) (color 0 0 0 0)
