File: power.kicad_sch (KiCad schematic)
At the start: 22 parts, among them U2 AP62150WU, U4 TLV75533PDBV, U5 USBLC6-2SC6

Commit message: Fix revision
Parts:
- U4: Mouser Part Number (none) -> 595-TLV75533PDBVR
- U5: Mouser Part Number (none) -> 511-USBLC6-2SC6
Other:
- title: openautolab - Mainboard -> openautolab - Alternative Mainboard
Changed lines of the file:
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@@
   (paper "A4")
   (title_block
-    (title "openautolab - Mainboard")
+    (title "openautolab - Alternative Mainboard")
     (date "2024-04-03")
-    (rev "2.0")
+    (rev "1")
   )
   (junction (at 207.645 127) (diameter 0) (color 0 0 0 0)
@@
     (property "Datasheet" "https://www.st.com/resource/en/datasheet/usblc6-2.pdf" (at 258.445 67.31 0)
       (effects (font (size 1.27 1.27)) (justify left) hide)
+    )
+    (property "Mouser Part Number" "511-USBLC6-2SC6 " (at 257.175 59.055 0)
+      (effects (font (size 1.27 1.27)) hide)
     )
     (pin "5")
@@
       (effects (font (size 1.27 1.27)) hide)
     )
+    (property "Mouser Part Number" "595-TLV75533PDBVR " (at 219.075 129.54 0)
+      (effects (font (size 1.27 1.27)) hide)
+    )
