File: mainboard.kicad_pcb (KiCad board)
At the start: 4 copper layers, 150 x 70 mm, 101 parts, among them J1 HX711, J10 MainPump, J11 WaterLevelSensor, J12 AuxPump, J13 OneWireTemp, J14 OneWireTemp, J15 FlowSensor, J16 DC 12V IN, J17 USB_C_Receptacle_USB2.0_16P, J18 Conn_01x14_MountingPin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

Commit message: Fix revision on board
Other:
- board text added: "openautolab alternative mainboard rev. 2"
- board text removed: "openautolab alternative mainboard rev. 1"
